Commit message: Updated update_windows_urdf.py to only flip forward slashes within quotation marks to backward slashes. Ran that script and flipped the slashes of robot.urdf

File: urdf/robot.urdf (robot description, URDF)
Before this commit: robot servobot, 13 links, 12 joints
Links:
- link 2000_0025_0002: geometry collision mesh filename=package:\\servobot_description\meshes\2000_0025_0002.stl; collision mesh filename=package:\\servobot_description\meshes\mg995_gear2.stl
- link 2000_0025_0002_2: geometry collision mesh filename=package:\\servobot_description\meshes\2000_0025_0002.stl; collision mesh filename=package:\\servobot_description\meshes\mg995_gear2.stl
- link 2000_0025_0002_3: geometry collision mesh filename=package:\\servobot_description\meshes\2000_0025_0002.stl; collision mesh filename=package:\\servobot_description\meshes\mg995_gear2.stl
- link 2000_0025_0002_4: geometry collision mesh filename=package:\\servobot_description\meshes\2000_0025_0002.stl; collision mesh filename=package:\\servobot_description\meshes\mg995_gear2.stl
- link chassisasm: mass 1.00595 -> 1.41284; geometry collision mesh filename=package:\\servobot_description\meshes\2000_0025_0002.stl; collision mesh filename=package:\\servobot_description\meshes\2000_0025_0002.stl
- link hipasm: geometry collision mesh filename=package:\\servobot_description\meshes\2000_0025_0002.stl; collision mesh filename=package:\\servobot_description\meshes\2000_0025_0002__2.stl
- link hipasm_2: geometry collision mesh filename=package:\\servobot_description\meshes\2000_0025_0002.stl; collision mesh filename=package:\\servobot_description\meshes\2000_0025_0002__2.stl
- link hipasm_3: geometry collision mesh filename=package:\\servobot_description\meshes\2000_0025_0002.stl; collision mesh filename=package:\\servobot_description\meshes\2000_0025_0002__2.stl
- link hipasm_4: geometry collision mesh filename=package:\\servobot_description\meshes\2000_0025_0002.stl; collision mesh filename=package:\\servobot_description\meshes\2000_0025_0002__2.stl
- link part_1: geometry collision mesh filename=package:\\servobot_description\meshes\2000_0025_0002__2.stl; collision mesh filename=package:\\servobot_description\meshes\mg995_gear2.stl
- link part_1_2: geometry collision mesh filename=package:\\servobot_description\meshes\2000_0025_0002__2.stl; collision mesh filename=package:\\servobot_description\meshes\mg995_gear2.stl
- link part_1_3: geometry collision mesh filename=package:\\servobot_description\meshes\2000_0025_0002__2.stl; collision mesh filename=package:\\servobot_description\meshes\mg995_gear2.stl
- link part_1_4: geometry collision mesh filename=package:\\servobot_description\meshes\2000_0025_0002__2.stl; collision mesh filename=package:\\servobot_description\meshes\mg995_gear2.stl
Joints:
- joint bl_bot: limit lower=-1.5708 upper=1.5708 effort=2.1 velocity=6.5 -> lower=-1.5708 upper=1.5708 effort=10 velocity=10
- joint bl_hip: limit lower=-0.523599 upper=0.523599 effort=2.1 velocity=6.5 -> lower=-1 upper=1 effort=10 velocity=10
- joint bl_top: limit lower=-1.5708 upper=1.5708 effort=2.1 velocity=6.5 -> lower=-1.5708 upper=1.5708 effort=10 velocity=10
- joint br_bot: limit lower=-1.5708 upper=1.5708 effort=2.1 velocity=6.5 -> lower=-1.5708 upper=1.5708 effort=10 velocity=10
- joint br_hip: limit lower=-0.523599 upper=0.523599 effort=2.1 velocity=6.5 -> lower=-1 upper=1 effort=10 velocity=10
- joint br_top: limit lower=-1.5708 upper=1.5708 effort=2.1 velocity=6.5 -> lower=-1.5708 upper=1.5708 effort=10 velocity=10
- joint fl_bot: limit lower=-1.5708 upper=1.5708 effort=2.1 velocity=6.5 -> lower=-1.5708 upper=1.5708 effort=10 velocity=10
- joint fl_hip: limit lower=-0.523599 upper=0.523599 effort=2.1 velocity=6.5 -> lower=-1 upper=1 effort=10 velocity=10
- joint fl_top: limit lower=-1.5708 upper=1.5708 effort=2.1 velocity=6.5 -> lower=-1.5708 upper=1.5708 effort=10 velocity=10
- joint fr_bot: limit lower=-1.5708 upper=1.5708 effort=2.1 velocity=6.5 -> lower=-1.5708 upper=1.5708 effort=10 velocity=10
- joint fr_hip: limit lower=-0.523599 upper=0.523599 effort=2.1 velocity=6.5 -> lower=-1 upper=1 effort=10 velocity=10
- joint fr_top: limit lower=-1.5708 upper=1.5708 effort=2.1 velocity=6.5 -> lower=-1.5708 upper=1.5708 effort=10 velocity=10
